File: Documentation/entity_system/entity_module.sch (EAGLE design)
At the start: 200 parts, among them IC1 74LS14N, IC2 74LS14N, IC3 74LS14N, IC4 74LS14N, IC5 74LS14N, IC6 74LS14N, IC7 74LS14N, M1 CD74HCT151E, M2 CD74HCT151E, M3 CD74HCT151E, M4 CD74HCT151E, M5 CD74HCT151E, Q1 16MHZ, T1 BJT, T10 2N3565, T11 2N3565, T12 2N3565, T13 2N3565, T14 2N3565, T15 2N3565, T16 2N3565, T17 2N3565, T18 2N3565, T19 2N3565, T2 BJT, T20 2N3565, T21 2N3565, T22 2N3565, T23 2N3565, T24 2N3565, T25 2N3565, T26 2N3565, T27 2N3565, T28 2N3565, T29 2N3565, T3 BJT, T30 2N3565, T31 2N3565, T32 2N3565, T33 2N3565, T34 2N3565, T35 2N3565, T36 2N3565, T37 2N3565, T38 2N3565, T39 2N3565, T4 BJT, T40 2N3565, T41 2N3565, T42 2N3565, T43 2N3565, T44 2N3565, T5 2N3565, T6 2N3565, T7 2N3565, T8 2N3565, T9 2N3565, X1 22-23-2021, X10 22-23-2021, X11 22-23-2021, X12 22-23-2021, X13 22-23-2021, X14 22-23-2021, X15 22-23-2021, X16 22-23-2021, X17 22-23-2021, X18 22-23-2021, X19 22-23-2021, X2 22-23-2021, X20 22-23-2021, X21 22-23-2021, X22 22-23-2021, X23 22-23-2021, X24 22-23-2021, X25 22-23-2021, X26 22-23-2021, X27 22-23-2021, X28 22-23-2021, X29 22-23-2021, X3 22-23-2021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

Commit message: Added PSU and entity module schematic
Parts:
- removed C10, C11, C12, C13, C16, C17, C18, C19, C20, C21, C22, C23, C24, C25, C26, C27, C28, C29, C30, C31, C32, C33, C34, C35, C36, C37, C38, C39, C40, C41, C42, C43, C44, C45, C46, C47, C6, C7, C8, C9: 0.1uF, rcl:C-US025-024X044
- removed IC1, IC2, IC3, IC4, IC5, IC6, IC7: 74LS14N, 74xx-us:74LS14N
- removed M1, M2, M3, M4, M5: CD74HCT151E, Custom:CD74HCT151E
- removed POWER1, X1, X10, X11, X12, X13, X14, X15, X16, X17, X18, X19, X2, X20, X21, X22, X23, X24, X25, X26, X27, X28, X29, X3, X30, X31, X32, X33, X34, X35, X36, X37, X38, X39, X4, X40, X5, X6, X7, X8, X9: 22-23-2021, con-molex:22-23-2021
- removed R10, R11, R12, R13, R14, R15, R17, R18, R19, R20, R21, R22, R23, R24, R25, R26, R27, R28, R29, R30, R31, R32, R33, R34, R35, R36, R37, R38, R39, R40, R41, R42, R43, R44, R45, R46, R47, R48, R8, R9: 10KOHM, rcl:R-US_0204/7
- removed T10, T11, T12, T13, T14, T15, T16, T17, T18, T19, T20, T21, T22, T23, T24, T25, T26, T27, T28, T29, T30, T31, T32, T33, T34, T35, T36, T37, T38, T39, T40, T41, T42, T43, T44, T5, T6, T7, T8, T9: 2N3565, transistor:2N3565
- added IR: 22-23-2041, con-molex:22-23-2041
- added SERVO: 22-23-2031, con-molex:22-23-2031
Connections:
- removed net D1: IC1A.O, M1.I0
- removed net D10: IC2D.O, M3.I1
- removed net D11: IC2E.O, M1.I2
- removed net D12: IC2F.O, M4.I2
- removed net D13: IC3A.O, M2.I2
- removed net D14: IC3B.O, M5.I2
- removed net D15: IC3C.O, M3.I2
- removed net D16: IC3D.O, M1.I3
- removed net D17: IC3E.O, M4.I3
- removed net D18: IC3F.O, M2.I3
- removed net D19: IC4A.O, M5.I3
- removed net D2: IC1B.O, M4.I0
- removed net D20: IC4B.O, M3.I3
- removed net D21: IC4C.O, M1.I4
- removed net D22: IC4D.O, M4.I4
- removed net D23: IC4E.O, M2.I4
- removed net D24: IC4F.O, M5.I4
- removed net D25: IC5A.O, M3.I4
- removed net D26: IC5B.O, M1.I5
- removed net D27: IC5C.O, M4.I5
- removed net D28: IC5D.O, M2.I5
- removed net D29: IC5E.O, M5.I5
- removed net D3: IC1C.O, M2.I0
- removed net D30: IC5F.O, M3.I5
- removed net D31: IC6A.O, M1.I6
- removed net D32: IC6B.O, M4.I6
- removed net D33: IC6C.O, M2.I6
- removed net D34: IC6D.O, M5.I6
- removed net D35: IC6E.O, M3.I6
- removed net D36: IC6F.O, M1.I7
- removed net D37: IC7A.O, M4.I7
- removed net D38: IC7B.O, M2.I7
- removed net D39: IC7C.O, M5.I7
- removed net D4: IC1D.O, M5.I0
- removed net D40: IC7D.O, M3.I7
- removed net D5: IC1E.O, M3.I0
- removed net D6: IC1F.O, M1.I1
- removed net D7: IC2A.O, M4.I1
- removed net D8: IC2B.O, M2.I1
- removed net D9: IC2C.O, M5.I1
- removed net N$10: T14.C, X31-2.S
- removed net N$11: T15.C, X30-2.S
- removed net N$12: T16.C, X29-2.S
- removed net N$13: T17.C, X28-2.S
- removed net N$14: T18.C, X27-2.S
- removed net N$15: T19.C, X26-2.S
- removed net N$16: T20.C, X25-2.S
- removed net N$17: T21.C, X24-2.S
- removed net N$18: T22.C, X23-2.S
- removed net N$19: T23.C, X22-2.S
- removed net N$2: T6.C, X39-2.S
- removed net N$20: T24.C, X21-2.S
- removed net N$21: T25.C, X20-2.S
- removed net N$22: T26.C, X19-2.S
- removed net N$23: T27.C, X18-2.S
- removed net N$24: T28.C, X17-2.S
- removed net N$25: T29.C, X16-2.S
- removed net N$26: T30.C, X15-2.S
- removed net N$27: T31.C, X14-2.S
- removed net N$28: T32.C, X13-2.S
- removed net N$29: T33.C, X12-2.S
- removed net N$3: T7.C, X38-2.S
- removed net N$30: T34.C, X11-2.S
- removed net N$31: T35.C, X10-2.S
- removed net N$32: T36.C, X9-2.S
- removed net N$33: T37.C, X8-2.S
- removed net N$34: T38.C, X7-2.S
- removed net N$35: T39.C, X6-2.S
- removed net N$36: T40.C, X5-2.S
- removed net N$37: T41.C, X4-2.S
- removed net N$38: T42.C, X3-2.S
- removed net N$39: T43.C, X2-2.S
- removed net N$4: T8.C, X37-2.S
- removed net N$40: T44.C, X1-2.S
- removed net N$5: T9.C, X36-2.S
- removed net N$6: T10.C, X35-2.S
- removed net N$7: T11.C, X34-2.S
- removed net N$8: T12.C, X33-2.S
- removed net N$9: T13.C, X32-2.S
- removed net RESULT1: ATMEGA.4, M1.Y
- removed net RESULT2: ATMEGA.5, M4.Y
- removed net RESULT3: ATMEGA.6, M2.Y
- removed net RESULT4: ATMEGA.13, M5.Y
- removed net RESULT5: ATMEGA.14, M3.Y
- removed net SELECT1: ATMEGA.11, M1.S0, M2.S0, M3.S0, M4.S0, M5.S0, M5.S1
- removed net SELECT2: ATMEGA.12, M1.S1, M2.S1, M3.S1, M3.S2, M4.S1
- removed net SELECT3: ATMEGA.15, M1.S2, M2.S2, M4.S2, M5.S2
- removed net SELECT4: ATMEGA.16, M1.E', M1.GND, M2.E', M2.GND, M3.E', M3.GND, M4.E', M4.GND, M5.E', M5.GND
- removed net SELECT5: ATMEGA.17, T10.B, T11.B, T12.B, T13.B, T14.B, T15.B, T16.B, T17.B, T18.B, T19.B, T20.B, T21.B, T22.B, T23.B, T24.B, T25.B, T26.B, T27.B, T28.B, T29.B, T30.B, T31.B, T32.B, T33.B, T34.B, T35.B, T36.B, T37.B, T38.B, T39.B, T40.B, T41.B, T42.B, T43.B, T44.B, T5.B, T6.B, T7.B, T8.B, T9.B
- removed net W1: C6.1, IC1A.I, R8.2, T5.E
- removed net W10: C17.1, IC2D.I, R18.2, T14.E
- removed net W11: C18.1, IC2E.I, R19.2, T15.E
- removed net W12: C19.1, IC2F.I, R20.2, T16.E
- removed net W13: C20.1, IC3A.I, R21.2, T17.E
- removed net W14: C21.1, IC3B.I, R22.2, T18.E
- removed net W15: C22.1, IC3C.I, R23.2, T19.E
- removed net W16: C23.1, IC3D.I, R24.2, T20.E
- removed net W17: C24.1, IC3E.I, R25.2, T21.E
- removed net W18: C25.1, IC3F.I, R26.2, T22.E
- removed net W19: C26.1, IC4A.I, R27.2, T23.E
- removed net W2: C7.1, IC1B.I, R9.2, T6.E
- removed net W20: C27.1, IC4B.I, R28.2, T24.E
- removed net W21: C28.1, IC4C.I, R29.2, T25.E
- removed net W22: C29.1, IC4D.I, R30.2, T26.E
- removed net W23: C30.1, IC4E.I, R31.2, T27.E
- removed net W24: C31.1, IC4F.I, R32.2, T28.E
- removed net W25: C32.1, IC5A.I, R33.2, T29.E
- removed net W26: C33.1, IC5B.I, R34.2, T30.E
- removed net W27: C34.1, IC5C.I, R35.2, T31.E
- removed net W28: C35.1, IC5D.I, R36.2, T32.E
- removed net W29: C36.1, IC5E.I, R37.2, T33.E
- removed net W3: C8.1, IC1C.I, R10.2, T7.E
- removed net W30: C37.1, IC5F.I, R38.2, T34.E
- removed net W31: C38.1, IC6A.I, R39.2, T35.E
- removed net W32: C39.1, IC6B.I, R40.2, T36.E
- removed net W33: C40.1, IC6C.I, R41.2, T37.E
- removed net W34: C41.1, IC6D.I, R42.2, T38.E
- removed net W35: C42.1, IC6E.I, R43.2, T39.E
- removed net W36: C43.1, IC6F.I, R44.2, T40.E
- removed net W37: C44.1, IC7A.I, R45.2, T41.E
- removed net W38: C45.1, IC7B.I, R46.2, T42.E
- removed net W39: C46.1, IC7C.I, R47.2, T43.E
- removed net W4: C9.1, IC1D.I, R11.2, T8.E
- removed net W40: C47.1, IC7D.I, R48.2, T44.E
- removed net W5: C10.1, IC1E.I, R12.2, T9.E
- removed net W6: C11.1, IC1F.I, R13.2, T10.E
- removed net W7: C12.1, IC2A.I, R14.2, T11.E
- removed net W8: C13.1, IC2B.I, R15.2, T12.E
- removed net W9: C16.1, IC2C.I, R17.2, T13.E
- new net OPTION10: ATMEGA.13
- new net OPTION11: ATMEGA.14
- new net OPTION12: ATMEGA.15
- new net OPTION13: ATMEGA.16
- new net OPTION14: ATMEGA.17
- new net OPTION6: ATMEGA.4
- new net OPTION7: ATMEGA.6
- new net OPTION8: ATMEGA.11
- new net OPTION9: ATMEGA.12
- net 5V: now also IR-2.S, SERVO-2.S; no longer IC1P.VCC, IC2P.VCC, IC3P.VCC, IC4P.VCC, IC5P.VCC, IC6P.VCC, IC7P.VCC, M1.VCC, M2.VCC, M3.VCC, M4.VCC, M5.VCC, POWER1-2.S, R10.1, R11.1, R12.1, R13.1, R14.1, R15.1, R17.1, R18.1, R19.1, R20.1, R21.1, R22.1, R23.1, R24.1, R25.1, R26.1, R27.1, R28.1, R29.1, R30.1, R31.1, R32.1, R33.1, R34.1, R35.1, R36.1, R37.1, R38.1, R39.1, R40.1, R41.1, R42.1, R43.1, R44.1, R45.1, R46.1, R47.1, R48.1, R8.1, R9.1
- net GND: now also IR-1.S, SERVO-1.S; no longer C10.2, C11.2, C12.2, C13.2, C16.2, C17.2, C18.2, C19.2, C20.2, C21.2, C22.2, C23.2, C24.2, C25.2, C26.2, C27.2, C28.2, C29.2, C30.2, C31.2, C32.2, C33.2, C34.2, C35.2, C36.2, C37.2, C38.2, C39.2, C40.2, C41.2, C42.2, C43.2, C44.2, C45.2, C46.2, C47.2, C6.2, C7.2, C8.2, C9.2, IC1P.GND, IC2P.GND, IC3P.GND, IC4P.GND, IC5P.GND, IC6P.GND, IC7P.GND, POWER1-1.S, X1-1.S, X10-1.S, X11-1.S, X12-1.S, X13-1.S, X14-1.S, X15-1.S, X16-1.S, X17-1.S, X18-1.S, X19-1.S, X2-1.S, X20-1.S, X21-1.S, X22-1.S, X23-1.S, X24-1.S, X25-1.S, X26-1.S, X27-1.S, X28-1.S, X29-1.S, X3-1.S, X30-1.S, X31-1.S, X32-1.S, X33-1.S, X34-1.S, X35-1.S, X36-1.S, X37-1.S, X38-1.S, X39-1.S, X4-1.S, X40-1.S, X5-1.S, X6-1.S, X7-1.S, X8-1.S, X9-1.S
- net N$1: now also ATMEGA.5, SERVO-3.S; no longer T5.C, X40-2.S
- net SCL-5V: now also IR-4.S
- net SDA-5V: now also IR-3.S
Other:
- note added: "1.0"
- note removed: "1.3"
- note removed: "W1"
